File: hardware/Node/Node.brd (EAGLE design)
At the start: 49.5 x 49.5 mm, 71 parts, among them J1 AVR_SPI_PRG_6NS, J2 M04X2, Q1 PMR280UN, Q2 PMR280UN, Q3 PMR280UN, SW1 KSS, SW2 KSS, U1 ATMEGA32U4QFN, U2 BLUETOOTH-RN41", U3 LSM303DLM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

Commit message: Add labels
Parts:
- added OSHW: (no value), ohw-logo:OSHW_FILLX200_NOTEXT
Other:
- board text added: "3V3"
- board text added: "AVR ISP"
- board text added: "Adjacent"
- board text added: "Adjacent Reality Node 0.1"
- board text added: "BT_R"
- board text added: "Creative Commons BY-SA 3.0"
- board text added: "Donald Cober & Nirav Patel"
- board text added: "F0"
- board text added: "F1"
- board text added: "F4"
- board text added: "F5"
- board text added: "F6"
- board text added: "F7"
- board text added: "GND"
- board text added: "HWB"
- board text added: "Node 0.1"
- board text added: "POWER"
- board text added: "RESET"
- board text added: "RXI"
- board text added: "Reality"
- board text added: "SW1"
- board text added: "SW2"
- board text added: "TXO"
- board text added: "VBUS"
- board text added: "VIN"
- board text added: "X"
- board text added: "Y"
- board text added: "Z"
- board text added: "http://adjacentreality.org"
- board text added: "https://github.com/dcoberii/"
Changed lines of the file:
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@@
 <layer number="27" name="tValues" color="7" fill="1" visible="yes" active="yes"/>
 <layer number="28" name="bValues" color="7" fill="1" visible="yes" active="yes"/>
-<layer number="29" name="tStop" color="7" fill="3" visible="no" active="yes"/>
-<layer number="30" name="bStop" color="7" fill="6" visible="no" active="yes"/>
+<layer number="29" name="tStop" color="7" fill="3" visible="yes" active="yes"/>
+<layer number="30" name="bStop" color="7" fill="6" visible="yes" active="yes"/>
 <layer number="31" name="tCream" color="7" fill="4" visible="no" active="yes"/>
 <layer number="32" name="bCream" color="7" fill="5" visible="no" active="yes"/>
@@
 <layer number="123" name="tTestmark" color="7" fill="1" visible="no" active="yes"/>
 <layer number="124" name="bTestmark" color="7" fill="1" visible="no" active="yes"/>
-<layer number="125" name="_tNames" color="7" fill="1" visible="no" active="yes"/>
+<layer number="125" name="_tNames" color="7" fill="1" visible="yes" active="yes"/>
 <layer number="126" name="_bNames" color="7" fill="1" visible="yes" active="yes"/>
 <layer number="127" name="_tValues" color="7" fill="1" visible="yes" active="yes"/>
@@
 <rectangle x1="6.985" y1="34.29" x2="15.875" y2="49.53" layer="40"/>
 <rectangle x1="6.985" y1="34.29" x2="15.875" y2="49.53" layer="42"/>
+<text x="18.415" y="35.8775" size="1.27" layer="21" font="vector" rot="R90">VBUS</text>
+<text x="20.955" y="35.8775" size="1.27" layer="21" font="vector" rot="R90">3V3</text>
+<text x="23.495" y="35.8775" size="1.27" layer="21" font="vector" rot="R90">VIN</text>
+<text x="26.035" y="35.8775" size="1.27" layer="21" rot="R90">RXI</text>
+<text x="28.575" y="35.8775" size="1.27" layer="21" font="vector" rot="R90">TXO</text>
+<text x="31.115" y="35.8775" size="1.27" layer="21" font="vector" rot="R90">GND</text>
+<text x="48.895" y="29.845" size="1.27" layer="21" font="vector" rot="R90">GND</text>
+<text x="46.355" y="29.845" size="1.27" layer="21" font="vector" rot="R90">3V3</text>
+<text x="44.45" y="19.685" size="1.27" layer="21" font="vector" rot="R90">F7</text>
+<text x="42.545" y="19.685" size="1.27" layer="21" font="vector" rot="R90">F6</text>
+<text x="44.45" y="22.225" size="1.27" layer="21" font="vector" rot="R90">F5</text>
+<text x="42.545" y="22.225" size="1.27" layer="21" font="vector" rot="R90">F4</text>
+<text x="44.45" y="24.765" size="1.27" layer="21" font="vector" rot="R90">F1</text>
+<text x="42.545" y="24.765" size="1.27" layer="21" font="vector" rot="R90">F0</text>
+<text x="45.72" y="41.275" size="1.27" layer="21" font="vector">SW2</text>
+<text x="45.72" y="16.51" size="1.27" layer="21" font="vector">SW1</text>
+<text x="0.3175" y="41.275" size="1.27" layer="21" font="vector">RESET</text>
+<text x="1.905" y="16.51" size="1.27" layer="21" font="vector">HWB</text>
+<text x="10.795" y="4.445" size="1.27" layer="21" font="vector">POWER</text>
+<text x="18.0975" y="31.115" size="1.27" layer="21" font="vector">BT_R</text>
+<text x="6.6675" y="20.955" size="1.27" layer="21" font="vector" rot="R90">AVR ISP</text>
+<wire x1="31.75" y1="25.4" x2="31.75" y2="20.32" width="0.254" layer="21"/>
+<wire x1="31.75" y1="25.4" x2="30.48" y2="24.13" width="0.254" layer="21"/>
+<wire x1="31.75" y1="25.4" x2="33.02" y2="24.13" width="0.254" layer="21"/>
+<wire x1="33.02" y1="19.05" x2="38.1" y2="19.05" width="0.254" layer="21"/>
+<wire x1="38.1" y1="19.05" x2="36.83" y2="20.32" width="0.254" layer="21"/>
+<wire x1="38.1" y1="19.05" x2="36.83" y2="17.78" width="0.254" layer="21"/>
+<circle x="36.83" y="24.13" radius="0.635" width="0.254" layer="21"/>
+<circle x="36.83" y="24.13" radius="0.127" width="0.254" layer="21"/>
+<text x="33.02" y="24.13" size="1.524" layer="21" font="vector">Y</text>
+<text x="38.1" y="19.05" size="1.524" layer="21" font="vector">X</text>
+<text x="38.1" y="24.13" size="1.524" layer="21" font="vector">Z</text>
+<text x="7.62" y="27.94" size="2.286" layer="21" font="vector">Adjacent</text>
+<text x="7.62" y="24.765" size="2.286" layer="21" font="vector">Reality</text>
+<text x="7.62" y="21.59" size="2.286" layer="21" font="vector">Node 0.1</text>
+<rectangle x1="10.16" y1="9.525" x2="40.64" y2="17.145" layer="22"/>
+<rectangle x1="10.16" y1="9.525" x2="17.78" y2="40.005" layer="22"/>
+<rectangle x1="33.02" y1="9.525" x2="40.64" y2="40.005" layer="22"/>
+<rectangle x1="10.16" y1="32.385" x2="40.64" y2="40.005" layer="22"/>
+<rectangle x1="17.78" y1="17.145" x2="21.59" y2="32.385" layer="22"/>
+<rectangle x1="21.59" y1="28.575" x2="33.02" y2="32.385" layer="22"/>
+<rectangle x1="21.59" y1="20.955" x2="25.4" y2="28.575" layer="22"/>
+<rectangle x1="25.4" y1="20.955" x2="29.21" y2="24.765" layer="22"/>
+<rectangle x1="29.21" y1="24.765" x2="33.02" y2="28.575" layer="22"/>
+<text x="41.91" y="45.72" size="1.524" layer="22" font="vector" rot="MR0">Adjacent Reality Node 0.1</text>
+<text x="41.91" y="43.18" size="1.524" layer="22" font="vector" rot="MR0">Donald Cober &amp; Nirav Patel</text>
+<text x="8.89" y="3.81" size="1.524" layer="22" font="vector" rot="SMR180">http://adjacentreality.org</text>
+<text x="8.89" y="6.35" size="1.524" layer="22" font="vector" rot="SMR180">https://github.com/dcoberii/</text>
+<text x="43.815" y="38.4175" size="1.27" layer="22" font="vector" rot="MR270">Creative Commons BY-SA 3.0</text>
 </plain>
 <attributes>
@@
 <element name="U$4" library="SparkFun" package="STAND-OFF-TIGHT" value="" x="46.355" y="3.175"/>
 <element name="JP2" library="SparkFun" package="1X06" value="" x="17.78" y="41.91"/>
+<element name="OSHW" library="ohw-logo" package="OSHW_FILLX200_NOTEXT" value="" x="7.62" y="38.1" rot="MR270"/>
 </elements>
 <signals>
